Commit message: managed to get the block in gazebo TO DO: Fix robot controller nodes not spawning

File: rgmc/src/pose_estimation/src/camera_model.xacro (robot description, xacro)
@@ -1,29 +1,58 @@
 <?xml version="1.0"?>
-<robot xmlns:xacro="http://wiki.ros.org/xacro" name="ur5e_robot">
-    <link name="camera_link">
-        <visual>
-            <geometry>
-                <box size="0.05 0.05 0.05" />
-            </geometry>
-            <material name="red" />
-        </visual>
-        <collision>
-            <geometry>
-                <box size="0.05 0.05 0.05" />
-            </geometry>
-        </collision>
-        <inertial>
-            <mass value="0.1" />
-            <origin xyz="0 0 0" rpy="0 0 0" />
-            <inertia
-                ixx="0.0001" ixy="0.0" ixz="0.0"
-                iyy="0.0001" iyz="0.0"
-                izz="0.0001" />
-        </inertial>
-    </link>
-    <joint name="camera_joint" type="fixed">
-        <parent link="tool0"/>
-        <child link="camera_link"/>
-        <origin xyz="0 0 0.1" rpy="0 0 0"/>
-    </joint>
+<robot xmlns:xacro="http://wiki.ros.org/xacro" name="camera_model">
+  <link name="camera_link">
+    <visual>
+      <geometry>
+        <box size="0.1 0.1 0.1"/>
+      </geometry>
+      <material name="red">
+        <color rgba="1.0 0.0 0.0 1.0"/>
+      </material>
+    </visual>
+    <collision>
+      <geometry>
+        <box size="5 5 5" />
+      </geometry>
+    </collision>
+    <inertial>
+      <mass value="0.0" />
+      <origin xyz="0 0 0" rpy="0 0 0" />
+      <inertia
+        ixx="0.000" ixy="0.0" ixz="0.0"
+        iyy="0.000" iyz="0.0"
+        izz="0.000" />
+    </inertial>
+  </link>
+  <joint name="camera_joint" type="fixed">
+    <parent link="tool0"/>
+    <child link="camera_link"/>
+    <origin xyz="0 0 0.1" rpy="0 0 0"/>
+  </joint>
+  <gazebo>
+    <sensor type="depth" name="depth_camera">
+      <always_on>true</always_on>
+      <update_rate>30.0</update_rate>
+      <camera>
+        <horizontal_fov>1.047</horizontal_fov>
+        <image>
+          <width>640</width>
+          <height>480</height>
+          <format>R8G8B8</format>
+        </image>
+        <clip>
+          <near>0.1</near>
+          <far>5.0</far>
+        </clip>
+      </camera>
+      <plugin name="camera_controller" filename="libgazebo_ros_openni_kinect.so">
+        <alwaysOn>true</alwaysOn>
+        <updateRate>0.0</updateRate>
+        <cameraName>depth_camera</cameraName>
+        <imageTopicName>depth/image_raw</imageTopicName>
+        <depthImageTopicName>depth/depth_image_raw</depthImageTopicName>
+        <cameraInfoTopicName>depth/camera_info</cameraInfoTopicName>
+        <frameName>camera_link</frameName>
+      </plugin>
+    </sensor>
+  </gazebo>
 </robot>
