Commit message: added gazebo file TODO: Figure out how to use pcl with realsense camera Current realsense repo only uses depth, not pointcloud

File: rgmc/src/pose_estimation/urdf/ur5e_camera.xacro (robot description, xacro)
@@ -362,5 +362,5 @@
     <!-- Define d435i sensor -->
     <xacro:sensor_d435 name="camera" topics_ns="camera" parent="tool0">
-        <origin xyx="0 0 0" rpy="0 0 0"/>
+        <origin xyz="0 -0.035 -0.03" rpy="0 -1.5707 1.5707"/>
     </xacro:sensor_d435>
     <gazebo>
